File: ESP32.kicad_sch (KiCad schematic)
At the start: 1 part

Commit message: added i2c to io_protection
Parts:
- removed U1: ~, symbol astromech_symbols:YD-ESP32-S3
Changed lines of the file:
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@@
 	(generator_version "8.0")
 	(paper "A4")
-	(symbol
-		(lib_id "astromech_symbols:YD-ESP32-S3")
-		(at 124.46 63.5 0)
-		(unit 1)
-		(exclude_from_sim no)
-		(in_bom yes)
-		(on_board yes)
-		(dnp no)
-		(fields_autoplaced yes)
-		(property "Reference" "U1"
-			(at 144.78 49.53 0)
-			(effects
-				(font
-					(size 1.27 1.27)
-				)
-			)
-		)
-		(property "Value" "~"
-			(at 144.78 52.07 0)
-			(effects
-				(font
-					(size 1.27 1.27)
-				)
-			)
-		)
-		(property "Footprint" ""
-			(at 134.62 59.69 0)
-			(effects
-				(font
-					(size 1.27 1.27)
-				)
-				(hide yes)
-			)
-		)
-		(property "Datasheet" ""
-			(at 134.62 59.69 0)
-			(effects
-				(font
-					(size 1.27 1.27)
-				)
-				(hide yes)
-			)
-		)
-		(property "Description" ""
-			(at 134.62 59.69 0)
-			(effects
-				(font
-					(size 1.27 1.27)
-				)
-				(hide yes)
-			)
-		)
-		(pin "18"
-		)
-		(pin "8"
-		)
-		(pin "17"
-		)
-		(pin "22"
-		)
-		(pin "7"
-		)
-		(pin "16"
-		)
-		(pin "40"
-		)
-		(pin "5"
-		)
-		(pin "14"
-		)
-		(pin "19"
-		)
-		(pin "20"
-		)
-		(pin "6"
-		)
-		(pin "2"
-		)
-		(pin "4"
-		)
-		(pin "21"
-		)
-		(pin "1"
-		)
-		(pin "41"
-		)
-		(pin "43"
-		)
-		(pin "44"
-		)
-		(pin "30"
-		)
-		(pin "29"
-		)
-		(pin "34"
-		)
-		(pin "37"
-		)
-		(pin "36"
-		)
-		(pin "35"
-		)
-		(pin "39"
-		)
-		(pin "33"
-		)
-		(pin "23"
-		)
-		(pin "15"
-		)
-		(pin "9"
-		)
-		(pin "24"
-		)
-		(pin "28"
-		)
-		(pin "31"
-		)
-		(pin "26"
-		)
-		(pin "11"
-		)
-		(pin "12"
-		)
-		(pin "32"
-		)
-		(pin "25"
-		)
-		(pin "27"
-		)
-		(pin "42"
-		)
-		(pin "3"
-		)
-		(pin "13"
-		)
-		(pin "10"
-		)
-		(pin "38"
-		)
-		(instances
-			(project ""
-				(path "/3ed70c37-1dc6-4761-9813-fca49ce12494/dcd705a8-d3f6-4ba0-a933-c0adcd8c1729"
-					(reference "U1")
-					(unit 1)
-				)
-			)
-		)
-	)
 )
