File: ESP32.kicad_sch (KiCad schematic)
At the start: 11 parts, among them Q1 BSS138, Q2 BSS138

Commit message: moved power protection
Parts:
- removed Q1, Q2: BSS138, Package_TO_SOT_SMD:SOT-23, symbol Transistor_FET:BSS138
- removed R4, R5, R6, R7: R, symbol Device:R
Connections:
- net Vin renamed 5Vin
Other:
- added sheet Level Converter (level_converter.kicad_sch)
- added sheet Level Converter1 (level_converter.kicad_sch)
