File: voltage_monitoring.kicad_sch (KiCad schematic)
At the start: 4 parts, among them IC1 MAX11645EUA+

Commit message: moved voltage monitoring
Parts:
- removed D2: D_Zener, symbol Device:D_Zener
- removed IC1: MAX11645EUA+, SOP65P490X111-8N, symbol MAX11645EUA+:MAX11645EUA+
- removed R1, R2: R, symbol Device:R

Commit message: first try
Parts:
- added D1, D2, D3, D4, D5, D6, D7, D8: LD271, LED_THT:LED_D5.0mm_IRGrey, symbol LED:LD271

Commit message: added i2c to io_protection
Parts:
- removed D1, D2, D3, D4, D5, D6, D7, D8: LD271, LED_THT:LED_D5.0mm_IRGrey, symbol LED:LD271
