File: io_expander.kicad_sch (KiCad schematic)
At the start: 0 parts

Commit message: Updated IO Expander
Created bus input (SCL, SDA, INT) and bus output (PO{15:0}).
Using the  TCA9554 Low Voltage 8-Bit for I2C communication. The output of PO is tied to the VCC input and each address is configurable with solder jumpers being tied to either VCC or GND.
Parts:
- added JP2, JP4, JP5, JP6, JP7, JP8: SolderJumper_3_Open, symbol Jumper:SolderJumper_3_Open
- added U2, U3: TCA9554DW, Package_SO:SOIC-16W_7.5x10.3mm_P1.27mm, symbol Interface_Expansion:TCA9554DW
Connections:
- new net A0: JP2.2 (C), JP7.2 (C), U2.1 (A0), U3.1 (A0)
- new net A1: JP4.2 (C), JP6.2 (C), U2.2 (A1), U3.2 (A1)
- new net A2: JP5.2 (C), JP8.2 (C), U2.3 (A2), U3.3 (A2)
- new net GND: JP2.1 (A), JP4.1 (A), JP5.1 (A), JP6.1 (A), JP7.1 (A), JP8.1 (A), U2.8 (GND), U3.8 (GND)
- new net INT: U2.13 (~{INT}), U3.13 (~{INT})
- new net PO_0: U2.4 (P0)
- new net PO_1: U2.5 (P1)
- new net PO_10: U3.6 (P2)
- new net PO_11: U3.7 (P3)
- new net PO_12: U3.9 (P4)
- new net PO_13: U3.10 (P5)
- new net PO_14: U3.11 (P6)
- new net PO_15: U3.12 (P7)
- new net PO_2: U2.6 (P2)
- new net PO_3: U2.7 (P3)
- new net PO_4: U2.9 (P4)
- new net PO_5: U2.10 (P5)
- new net PO_6: U2.11 (P6)
- new net PO_7: U2.12 (P7)
- new net PO_8: U3.4 (P0)
- new net PO_9: U3.5 (P1)
- new net SCL: U2.14 (SCL), U3.14 (SCL)
- new net SDA: U2.15 (SDA), U3.15 (SDA)
- new net VCC: JP2.3 (B), JP4.3 (B), JP5.3 (B), JP6.3 (B), JP7.3 (B), JP8.3 (B), U2.16 (VDD), U3.16 (VDD)
Other:
- note added: "I2C Input"
